Commit message: working on URDF

File: src/ros2_ws/src/oxbot_description/urdf/oxbot.urdf.xacro (robot description, xacro)
@@ -3,13 +3,13 @@
     <link name="base_footprint"/>
     <link name="chassis_bottom_link">
-        <inertial>
+        <!--<inertial>
             <origin xyz="0 0 0.0575" rpy="0.0 0.0 0.0"/>
             <mass value="8"/>
             <inertia ixx="9.330733e-02" iyy="2.1713733e-01" izz="2.92811333e-01"/>
-        </inertial>
+        </inertial>-->
         <visual>
             <origin rpy="0 0 0" xyz="0 0 0"/>
             <geometry>
-                <mesh filename="package://oxbot_description/meshes/oxbot_chassis_bottom.stl"/>
+                <mesh filename="package://oxbot_description/meshes/oxbot_chassis_bottom.stl" scale="0.001 0.001 0.001"/>
             </geometry>
         </visual>
@@ -17,5 +17,5 @@
             <origin rpy="0 0 0" xyz="0 0 0"/>
             <geometry>
-                <mesh filename="package://oxbot_description/meshes/oxbot_chassis_bottom.STL"/>
+                <mesh filename="package://oxbot_description/meshes/oxbot_chassis_bottom.stl" scale="0.001 0.001 0.001"/>
             </geometry>
         </collision>
@@ -27,12 +27,12 @@
     </joint>
     <link name="wheel_front_right_link">
-        <inertial>
+        <!--<inertial>
             <mass value="3"/>
             <inertia ixx="6.7775e-01" iyy="6.7775e-01" izz="1.35375e-02"/>
-        </inertial>
+        </inertial>-->
         <visual>
-            <origin rpy="0 0 0" xyz="75 0 0"/>
+            <origin rpy="0 3.1415 0" xyz="0.075 0 0"/>
             <geometry>
-                <mesh filename="package://oxbot_description/meshes/oxbot_front_wheel.stl"/>
+                <mesh filename="package://oxbot_description/meshes/oxbot_front_wheel.stl" scale="0.001 0.001 0.001"/>
             </geometry>
         </visual>
@@ -40,5 +40,5 @@
             <origin xyz="0 0 0" rpy="0 0 0"/>
             <geometry>
-                <mesh filename="package://oxbot_description/meshes/oxbot_front_wheel.stl"/>
+                <mesh filename="package://oxbot_description/meshes/oxbot_front_wheel.stl" scale="0.001 0.001 0.001"/>
             </geometry>
         </collision>
@@ -48,5 +48,29 @@
         <child link="wheel_front_right_link"/>
         <axis xyz="1 0 0"/>
-        <origin rpy="0 0 0" xyz="-0.28 0.1325 0"/>
+        <origin rpy="0 0 0" xyz="0.28 0.1325 0.026"/>
+    </joint>
+    <link name="wheel_front_left_link">
+        <!--<inertial>
+            <mass value="3"/>
+            <inertia ixx="6.7775e-01" iyy="6.7775e-01" izz="1.35375e-02"/>
+        </inertial>-->
+        <visual>
+            <origin rpy="0 0 0" xyz="-0.075 0 0"/>
+            <geometry>
+                <mesh filename="package://oxbot_description/meshes/oxbot_front_wheel.stl" scale="0.001 0.001 0.001"/>
+            </geometry>
+        </visual>
+        <collision>
+            <origin xyz="0 0 0" rpy="0 0 0"/>
+            <geometry>
+                <mesh filename="package://oxbot_description/meshes/oxbot_front_wheel.stl" scale="0.001 0.001 0.001"/>
+            </geometry>
+        </collision>
+    </link>
+    <joint name="wheel_front_left_joint" type="continuous">
+        <parent link="chassis_bottom_link"/>
+        <child link="wheel_front_left_link"/>
+        <axis xyz="1 0 0"/>
+        <origin rpy="0 0 0" xyz="-0.28 0.1325 0.026"/>
     </joint>
 </robot>

Commit message: updating URDF

File: src/ros2_ws/src/oxbot_description/urdf/oxbot.urdf.xacro (robot description, xacro)
@@ -74,3 +74,27 @@
         <origin rpy="0 0 0" xyz="-0.28 0.1325 0.026"/>
     </joint>
+    <link name="wheel_rear_right_link">
+        <!--<inertial>
+            <mass value="3"/>
+            <inertia ixx="6.7775e-01" iyy="6.7775e-01" izz="1.35375e-02"/>
+        </inertial>-->
+        <visual>
+            <origin rpy="0 3.1415 0" xyz="0.105 0 0"/>
+            <geometry>
+                <mesh filename="package://oxbot_description/meshes/oxbot_rear_wheel.stl" scale="0.001 0.001 0.001"/>
+            </geometry>
+        </visual>
+        <collision>
+            <origin xyz="0 0 0" rpy="0 0 0"/>
+            <geometry>
+                <mesh filename="package://oxbot_description/meshes/oxbot_rear_wheel.stl" scale="0.001 0.001 0.001"/>
+            </geometry>
+        </collision>
+    </link>
+    <joint name="wheel_rear_right_joint" type="continuous">
+        <parent link="chassis_bottom_link"/>
+        <child link="wheel_rear_right_link"/>
+        <axis xyz="1 0 0"/>
+        <origin rpy="0 0 0" xyz="0.28 -0.1325 0.049"/>
+    </joint>
 </robot>

Commit message: updating URDF

File: src/ros2_ws/src/oxbot_description/urdf/oxbot.urdf.xacro (robot description, xacro)
@@ -25,4 +25,28 @@
         <child link="chassis_bottom_link"/>
         <origin rpy="0 0 0" xyz="0 0 0.071"/>
+    </joint>
+    <link name="chassis_top_link">
+        <!--<inertial>
+            <origin xyz="0 0 0.0575" rpy="0.0 0.0 0.0"/>
+            <mass value="8"/>
+            <inertia ixx="9.330733e-02" iyy="2.1713733e-01" izz="2.92811333e-01"/>
+        </inertial>-->
+        <visual>
+            <origin rpy="0 0 0" xyz="0 0 0"/>
+            <geometry>
+                <mesh filename="package://oxbot_description/meshes/oxbot_chassis_top.stl" scale="0.001 0.001 0.001"/>
+            </geometry>
+        </visual>
+        <collision>
+            <origin rpy="0 0 0" xyz="0 0 0"/>
+            <geometry>
+                <mesh filename="package://oxbot_description/meshes/oxbot_chassis_top.stl" scale="0.001 0.001 0.001"/>
+            </geometry>
+        </collision>
+    </link>
+    <joint name="chassis_top_joint" type="fixed">
+        <parent link="chassis_bottom_link"/>
+        <child link="chassis_top_link"/>
+        <origin rpy="0 0 0" xyz="0 -0.0135 0.115"/>
     </joint>
     <link name="wheel_front_right_link">
@@ -98,3 +122,27 @@
         <origin rpy="0 0 0" xyz="0.28 -0.1325 0.049"/>
     </joint>
+    <link name="wheel_rear_left_link">
+        <!--<inertial>
+            <mass value="3"/>
+            <inertia ixx="6.7775e-01" iyy="6.7775e-01" izz="1.35375e-02"/>
+        </inertial>-->
+        <visual>
+            <origin rpy="0 0 0" xyz="-0.105 0 0"/>
+            <geometry>
+                <mesh filename="package://oxbot_description/meshes/oxbot_rear_wheel.stl" scale="0.001 0.001 0.001"/>
+            </geometry>
+        </visual>
+        <collision>
+            <origin xyz="0 0 0" rpy="0 0 0"/>
+            <geometry>
+                <mesh filename="package://oxbot_description/meshes/oxbot_rear_wheel.stl" scale="0.001 0.001 0.001"/>
+            </geometry>
+        </collision>
+    </link>
+    <joint name="wheel_rear_left_joint" type="continuous">
+        <parent link="chassis_bottom_link"/>
+        <child link="wheel_rear_left_link"/>
+        <axis xyz="1 0 0"/>
+        <origin rpy="0 0 0" xyz="-0.28 -0.1325 0.049"/>
+    </joint>
 </robot>

Commit message: updating URDF

File: src/ros2_ws/src/oxbot_description/urdf/oxbot.urdf.xacro (robot description, xacro)
@@ -49,4 +49,46 @@
         <child link="chassis_top_link"/>
         <origin rpy="0 0 0" xyz="0 -0.0135 0.115"/>
+    </joint>
+    <link name="camera_mount_link">
+        <!--<inertial>
+            <origin xyz="0 0 0.0575" rpy="0.0 0.0 0.0"/>
+            <mass value="8"/>
+            <inertia ixx="9.330733e-02" iyy="2.1713733e-01" izz="2.92811333e-01"/>
+        </inertial>-->
+        <visual>
+            <origin rpy="0 0 3.1415" xyz="0.09 0 0"/>
+            <geometry>
+                <mesh filename="package://oxbot_description/meshes/oxbot_realsense_mount.stl" scale="0.001 0.001 0.001"/>
+            </geometry>
+        </visual>
+        <collision>
+            <origin rpy="0 0 0" xyz="0 0 0"/>
+            <geometry>
+                <box size="0.180 0.03 0.04"/>
+            </geometry>
+        </collision>
+    </link>
+    <joint name="camera_mount_joint" type="fixed">
+        <parent link="chassis_top_link"/>
+        <child link="camera_mount_link"/>
+        <origin rpy="0 0 0" xyz="0 0.1075 0.140"/>
+    </joint>
+    <link name="camera_link">
+        <!--<inertial>
+            <origin xyz="0 0 0.0575" rpy="0.0 0.0 0.0"/>
+            <mass value="8"/>
+            <inertia ixx="9.330733e-02" iyy="2.1713733e-01" izz="2.92811333e-01"/>
+        </inertial>-->
+        <visual>
+            <origin rpy="1.57 0 3.1415" xyz="0 0.026 0"/>
+            <geometry>
+                <mesh filename="package://oxbot_description/meshes/d455.stl" scale="0.001 0.001 0.001"/>
+            </geometry>
+        </visual>
+    </link>
+    <joint name="camera_joint" type="fixed">
+        <parent link="camera_mount_link"/>
+        <child link="camera_link"/>
+        <origin rpy="0 0 0" xyz="0 -0.029 0.0325"/>
     </joint>
     <link name="wheel_front_right_link">

Commit message: added lidar to URDF

File: src/ros2_ws/src/oxbot_description/urdf/oxbot.urdf.xacro (robot description, xacro)
@@ -92,4 +92,28 @@
         <origin rpy="0 0 0" xyz="0 -0.029 0.0325"/>
     </joint>
+    <link name="lidar_link">
+        <!--<inertial>
+            <origin xyz="0 0 0.0575" rpy="0.0 0.0 0.0"/>
+            <mass value="8"/>
+            <inertia ixx="9.330733e-02" iyy="2.1713733e-01" izz="2.92811333e-01"/>
+        </inertial>-->
+        <visual>
+            <origin rpy="1.57 0 0" xyz="-0.0351 0.0351 -0.044"/>
+            <geometry>
+                <mesh filename="package://oxbot_description/meshes/rplidar_main.STL" scale="0.001 0.001 0.001"/>
+            </geometry>
+        </visual>
+        <collision>
+            <origin rpy="0 0 0" xyz="0 0 0"/>
+            <geometry>
+                <box size="0.110 0.09 0.09"/>
+            </geometry>
+        </collision>
+    </link>
+    <joint name="lidar_joint" type="fixed">
+        <parent link="chassis_top_link"/>
+        <child link="lidar_link"/>
+        <origin rpy="0 0 0" xyz="-0.01 0.015 0.184"/>
+    </joint>
     <link name="wheel_front_right_link">
         <!--<inertial>

Commit message: URDF collision updates

File: src/ros2_ws/src/oxbot_description/urdf/oxbot.urdf.xacro (robot description, xacro)
@@ -128,25 +128,73 @@
         </visual>
         <collision>
+            <origin xyz="0.075 0 0" rpy="0 0 0"/>
+            <geometry>
+                <mesh filename="package://oxbot_description/meshes/oxbot_front_wheel.stl" scale="0.001 0.001 0.001"/>
+            </geometry>
+        </collision>
+    </link>
+    <joint name="wheel_front_right_joint" type="continuous">
+        <parent link="chassis_bottom_link"/>
+        <child link="wheel_front_right_link"/>
+        <axis xyz="1 0 0"/>
+        <origin rpy="0 0 0" xyz="0.28 0.1325 0.026"/>
+    </joint>
+    <link name="wheel_front_left_link">
+        <!--<inertial>
+            <mass value="3"/>
+            <inertia ixx="6.7775e-01" iyy="6.7775e-01" izz="1.35375e-02"/>
+        </inertial>-->
+        <visual>
+            <origin rpy="0 0 0" xyz="-0.075 0 0"/>
+            <geometry>
+                <mesh filename="package://oxbot_description/meshes/oxbot_front_wheel.stl" scale="0.001 0.001 0.001"/>
+            </geometry>
+        </visual>
+        <collision>
+            <origin xyz="-0.075 0 0" rpy="0 0 0"/>
+            <geometry>
+                <mesh filename="package://oxbot_description/meshes/oxbot_front_wheel.stl" scale="0.001 0.001 0.001"/>
+            </geometry>
+        </collision>
+    </link>
+    <joint name="wheel_front_left_joint" type="continuous">
+        <parent link="chassis_bottom_link"/>
+        <child link="wheel_front_left_link"/>
+        <axis xyz="1 0 0"/>
+        <origin rpy="0 0 0" xyz="-0.28 0.1325 0.026"/>
+    </joint>
+    <link name="wheel_rear_right_link">
+        <!--<inertial>
+            <mass value="3"/>
+            <inertia ixx="6.7775e-01" iyy="6.7775e-01" izz="1.35375e-02"/>
+        </inertial>-->
+        <visual>
+            <origin rpy="0 3.1415 0" xyz="0.105 0 0"/>
+            <geometry>
+                <mesh filename="package://oxbot_description/meshes/oxbot_rear_wheel.stl" scale="0.001 0.001 0.001"/>
+            </geometry>
+        </visual>
+        <collision>
             <origin xyz="0 0 0" rpy="0 0 0"/>
             <geometry>
-                <mesh filename="package://oxbot_description/meshes/oxbot_front_wheel.stl" scale="0.001 0.001 0.001"/>
-            </geometry>
-        </collision>
-    </link>
-    <joint name="wheel_front_right_joint" type="continuous">
-        <parent link="chassis_bottom_link"/>
-        <child link="wheel_front_right_link"/>
-        <axis xyz="1 0 0"/>
-        <origin rpy="0 0 0" xyz="0.28 0.1325 0.026"/>
-    </joint>
-    <link name="wheel_front_left_link">
-        <!--<inertial>
-            <mass value="3"/>
-            <inertia ixx="6.7775e-01" iyy="6.7775e-01" izz="1.35375e-02"/>
-        </inertial>-->
-        <visual>
-            <origin rpy="0 0 0" xyz="-0.075 0 0"/>
-            <geometry>
-                <mesh filename="package://oxbot_description/meshes/oxbot_front_wheel.stl" scale="0.001 0.001 0.001"/>
+                <mesh filename="package://oxbot_description/meshes/oxbot_rear_wheel.stl" scale="0.001 0.001 0.001"/>
+            </geometry>
+        </collision>
+    </link>
+    <joint name="wheel_rear_right_joint" type="continuous">
+        <parent link="chassis_bottom_link"/>
+        <child link="wheel_rear_right_link"/>
+        <axis xyz="1 0 0"/>
+        <origin rpy="0 0 0" xyz="0.28 -0.1325 0.049"/>
+    </joint>
+    <link name="wheel_rear_left_link">
+        <!--<inertial>
+            <mass value="3"/>
+            <inertia ixx="6.7775e-01" iyy="6.7775e-01" izz="1.35375e-02"/>
+        </inertial>-->
+        <visual>
+            <origin rpy="0 0 0" xyz="-0.105 0 0"/>
+            <geometry>
+                <mesh filename="package://oxbot_description/meshes/oxbot_rear_wheel.stl" scale="0.001 0.001 0.001"/>
             </geometry>
         </visual>
@@ -154,52 +202,4 @@
             <origin xyz="0 0 0" rpy="0 0 0"/>
             <geometry>
-                <mesh filename="package://oxbot_description/meshes/oxbot_front_wheel.stl" scale="0.001 0.001 0.001"/>
-            </geometry>
-        </collision>
-    </link>
-    <joint name="wheel_front_left_joint" type="continuous">
-        <parent link="chassis_bottom_link"/>
-        <child link="wheel_front_left_link"/>
-        <axis xyz="1 0 0"/>
-        <origin rpy="0 0 0" xyz="-0.28 0.1325 0.026"/>
-    </joint>
-    <link name="wheel_rear_right_link">
-        <!--<inertial>
-            <mass value="3"/>
-            <inertia ixx="6.7775e-01" iyy="6.7775e-01" izz="1.35375e-02"/>
-        </inertial>-->
-        <visual>
-            <origin rpy="0 3.1415 0" xyz="0.105 0 0"/>
-            <geometry>
-                <mesh filename="package://oxbot_description/meshes/oxbot_rear_wheel.stl" scale="0.001 0.001 0.001"/>
-            </geometry>
-        </visual>
-        <collision>
-            <origin xyz="0 0 0" rpy="0 0 0"/>
-            <geometry>
-                <mesh filename="package://oxbot_description/meshes/oxbot_rear_wheel.stl" scale="0.001 0.001 0.001"/>
-            </geometry>
-        </collision>
-    </link>
-    <joint name="wheel_rear_right_joint" type="continuous">
-        <parent link="chassis_bottom_link"/>
-        <child link="wheel_rear_right_link"/>
-        <axis xyz="1 0 0"/>
-        <origin rpy="0 0 0" xyz="0.28 -0.1325 0.049"/>
-    </joint>
-    <link name="wheel_rear_left_link">
-        <!--<inertial>
-            <mass value="3"/>
-            <inertia ixx="6.7775e-01" iyy="6.7775e-01" izz="1.35375e-02"/>
-        </inertial>-->
-        <visual>
-            <origin rpy="0 0 0" xyz="-0.105 0 0"/>
-            <geometry>
-                <mesh filename="package://oxbot_description/meshes/oxbot_rear_wheel.stl" scale="0.001 0.001 0.001"/>
-            </geometry>
-        </visual>
-        <collision>
-            <origin xyz="0 0 0" rpy="0 0 0"/>
-            <geometry>
                 <mesh filename="package://oxbot_description/meshes/oxbot_rear_wheel.stl" scale="0.001 0.001 0.001"/>
             </geometry>

Commit message: added fans to URDF

File: src/ros2_ws/src/oxbot_description/urdf/oxbot.urdf.xacro (robot description, xacro)
@@ -116,4 +116,52 @@
         <origin rpy="0 0 0" xyz="-0.01 0.015 0.184"/>
     </joint>
+    <link name="fan1_link">
+        <!--<inertial>
+            <origin xyz="0 0 0.0575" rpy="0.0 0.0 0.0"/>
+            <mass value="8"/>
+            <inertia ixx="9.330733e-02" iyy="2.1713733e-01" izz="2.92811333e-01"/>
+        </inertial>-->
+        <visual>
+            <origin rpy="0 0 0" xyz="-0.121 0 0"/>
+            <geometry>
+                <mesh filename="package://oxbot_description/meshes/oxbot_fan.stl" scale="0.001 0.001 0.001"/>
+            </geometry>
+        </visual>
+        <collision>
+            <origin rpy="0 0 0" xyz="-0.121 0 0"/>
+            <geometry>
+                <mesh filename="package://oxbot_description/meshes/oxbot_fan.stl" scale="0.001 0.001 0.001"/>
+            </geometry>
+        </collision>
+    </link>
+    <joint name="fan1_joint" type="fixed">
+        <parent link="chassis_top_link"/>
+        <child link="fan1_link"/>
+        <origin rpy="0 0 0" xyz="0.215 -0.078 0.140"/>
+    </joint>
+    <link name="fan2_link">
+        <!--<inertial>
+            <origin xyz="0 0 0.0575" rpy="0.0 0.0 0.0"/>
+            <mass value="8"/>
+            <inertia ixx="9.330733e-02" iyy="2.1713733e-01" izz="2.92811333e-01"/>
+        </inertial>-->
+        <visual>
+            <origin rpy="0 0 0" xyz="-0.121 0 0"/>
+            <geometry>
+                <mesh filename="package://oxbot_description/meshes/oxbot_fan.stl" scale="0.001 0.001 0.001"/>
+            </geometry>
+        </visual>
+        <collision>
+            <origin rpy="0 0 0" xyz="-0.121 0 0"/>
+            <geometry>
+                <mesh filename="package://oxbot_description/meshes/oxbot_fan.stl" scale="0.001 0.001 0.001"/>
+            </geometry>
+        </collision>
+    </link>
+    <joint name="fan2_joint" type="fixed">
+        <parent link="chassis_top_link"/>
+        <child link="fan2_link"/>
+        <origin rpy="0 0 0" xyz="-0.085 -0.078 0.140"/>
+    </joint>
     <link name="wheel_front_right_link">
         <!--<inertial>

Commit message: added antenna to URDF

File: src/ros2_ws/src/oxbot_description/urdf/oxbot.urdf.xacro (robot description, xacro)
@@ -164,4 +164,23 @@
         <origin rpy="0 0 0" xyz="-0.085 -0.078 0.140"/>
     </joint>
+    <link name="antenna_link">
+        <visual>
+            <origin rpy="0 0 0" xyz="0 0 0"/>
+            <geometry>
+                <mesh filename="package://oxbot_description/meshes/oxbot_antenna.stl" scale="0.001 0.001 0.001"/>
+            </geometry>
+        </visual>
+        <collision>
+            <origin rpy="0 0 0" xyz="0 0 0"/>
+            <geometry>
+                <mesh filename="package://oxbot_description/meshes/oxbot_antenna.stl" scale="0.001 0.001 0.001"/>
+            </geometry>
+        </collision>
+    </link>
+    <joint name="antenna_joint" type="fixed">
+        <parent link="chassis_top_link"/>
+        <child link="antenna_link"/>
+        <origin rpy="0 0 0" xyz="0.068 -0.062 0.140"/>
+    </joint>
     <link name="wheel_front_right_link">
         <!--<inertial>
