Commit message: rotated oxbot to make +x forward

File: src/ros2_ws/src/oxbot_description/urdf/oxbot.urdf.xacro (robot description, xacro)
@@ -9,5 +9,5 @@
         </inertial>-->
         <visual>
-            <origin rpy="0 0 0" xyz="0 0 0"/>
+            <origin rpy="0 0 -1.57" xyz="0 0 0"/>
             <geometry>
                 <mesh filename="package://oxbot_description/meshes/oxbot_chassis_bottom.stl" scale="0.001 0.001 0.001"/>
@@ -33,5 +33,5 @@
         </inertial>-->
         <visual>
-            <origin rpy="0 0 0" xyz="0 0 0"/>
+            <origin rpy="0 0 -1.57" xyz="0 0 0"/>
             <geometry>
                 <mesh filename="package://oxbot_description/meshes/oxbot_chassis_top.stl" scale="0.001 0.001 0.001"/>
@@ -48,5 +48,5 @@
         <parent link="chassis_bottom_link"/>
         <child link="chassis_top_link"/>
-        <origin rpy="0 0 0" xyz="0 -0.0135 0.115"/>
+        <origin rpy="0 0 0" xyz="-0.0135 0 0.115"/>
     </joint>
     <link name="camera_mount_link">
@@ -57,5 +57,5 @@
         </inertial>-->
         <visual>
-            <origin rpy="0 0 3.1415" xyz="0.09 0 0"/>
+            <origin rpy="0 0 1.57" xyz="0 -0.09 0"/> <!--xyz="0.09 0 0"/> -->
             <geometry>
                 <mesh filename="package://oxbot_description/meshes/oxbot_realsense_mount.stl" scale="0.001 0.001 0.001"/>
@@ -72,5 +72,5 @@
         <parent link="chassis_top_link"/>
         <child link="camera_mount_link"/>
-        <origin rpy="0 0 0" xyz="0 0.1075 0.140"/>
+        <origin rpy="0 0 0" xyz="0.1075 0 0.140"/>
     </joint>
     <link name="camera_link">
@@ -81,5 +81,5 @@
         </inertial>-->
         <visual>
-            <origin rpy="1.57 0 3.1415" xyz="0 0.026 0"/>
+            <origin rpy="1.57 0 1.57" xyz="0 0 0"/>
             <geometry>
                 <mesh filename="package://oxbot_description/meshes/d455.stl" scale="0.001 0.001 0.001"/>
@@ -90,5 +90,5 @@
         <parent link="camera_mount_link"/>
         <child link="camera_link"/>
-        <origin rpy="0 0 0" xyz="0 -0.029 0.0325"/>
+        <origin rpy="0 0 0" xyz="-0.002 0 0.0325"/>
     </joint>
     <link name="lidar_link">
@@ -114,5 +114,5 @@
         <parent link="chassis_top_link"/>
         <child link="lidar_link"/>
-        <origin rpy="0 0 0" xyz="-0.01 0.015 0.184"/>
+        <origin rpy="0 0 -1.57" xyz="0.015 -0.01 0.184"/>
     </joint>
     <link name="fan1_link">
@@ -123,11 +123,11 @@
         </inertial>-->
         <visual>
-            <origin rpy="0 0 0" xyz="-0.121 0 0"/>
-            <geometry>
-                <mesh filename="package://oxbot_description/meshes/oxbot_fan.stl" scale="0.001 0.001 0.001"/>
-            </geometry>
-        </visual>
-        <collision>
-            <origin rpy="0 0 0" xyz="-0.121 0 0"/>
+            <origin rpy="0 0 0" xyz="0 0 0"/>
+            <geometry>
+                <mesh filename="package://oxbot_description/meshes/oxbot_fan.stl" scale="0.001 0.001 0.001"/>
+            </geometry>
+        </visual>
+        <collision>
+            <origin rpy="0 0 0" xyz="0 0 0"/>
             <geometry>
                 <mesh filename="package://oxbot_description/meshes/oxbot_fan.stl" scale="0.001 0.001 0.001"/>
@@ -138,5 +138,5 @@
         <parent link="chassis_top_link"/>
         <child link="fan1_link"/>
-        <origin rpy="0 0 0" xyz="0.215 -0.078 0.140"/>
+        <origin rpy="0 0 0" xyz="-.095 0.09 0.140"/>
     </joint>
     <link name="fan2_link">
@@ -147,11 +147,11 @@
         </inertial>-->
         <visual>
-            <origin rpy="0 0 0" xyz="-0.121 0 0"/>
-            <geometry>
-                <mesh filename="package://oxbot_description/meshes/oxbot_fan.stl" scale="0.001 0.001 0.001"/>
-            </geometry>
-        </visual>
-        <collision>
-            <origin rpy="0 0 0" xyz="-0.121 0 0"/>
+            <origin rpy="0 0 0" xyz="-0 0 0"/>
+            <geometry>
+                <mesh filename="package://oxbot_description/meshes/oxbot_fan.stl" scale="0.001 0.001 0.001"/>
+            </geometry>
+        </visual>
+        <collision>
+            <origin rpy="0 0 0" xyz="0 0 0"/>
             <geometry>
                 <mesh filename="package://oxbot_description/meshes/oxbot_fan.stl" scale="0.001 0.001 0.001"/>
@@ -162,5 +162,5 @@
         <parent link="chassis_top_link"/>
         <child link="fan2_link"/>
-        <origin rpy="0 0 0" xyz="-0.085 -0.078 0.140"/>
+        <origin rpy="0 0 0" xyz="-.095 -0.21 0.140"/>
     </joint>
     <link name="antenna_link">
@@ -181,5 +181,5 @@
         <parent link="chassis_top_link"/>
         <child link="antenna_link"/>
-        <origin rpy="0 0 0" xyz="0.068 -0.062 0.140"/>
+        <origin rpy="0 0 0" xyz="-0.057 -0.07 0.140"/>
     </joint>
     <link name="wheel_front_right_link">
@@ -189,5 +189,5 @@
         </inertial>-->
         <visual>
-            <origin rpy="0 3.1415 0" xyz="0.075 0 0"/>
+            <origin rpy="0 0 01.57" xyz="0 -0.075 0"/>
             <geometry>
                 <mesh filename="package://oxbot_description/meshes/oxbot_front_wheel.stl" scale="0.001 0.001 0.001"/>
@@ -201,9 +201,8 @@
         </collision>
     </link>
-    <joint name="wheel_front_right_joint" type="continuous">
+    <joint name="wheel_front_right_joint" type="fixed">
         <parent link="chassis_bottom_link"/>
         <child link="wheel_front_right_link"/>
-        <axis xyz="1 0 0"/>
-        <origin rpy="0 0 0" xyz="0.28 0.1325 0.026"/>
+        <origin rpy="0 0 0" xyz="0.1325 -0.28 0.026"/>
     </joint>
     <link name="wheel_front_left_link">
@@ -213,5 +212,5 @@
         </inertial>-->
         <visual>
-            <origin rpy="0 0 0" xyz="-0.075 0 0"/>
+            <origin rpy="0 0 -1.57" xyz="0 0.075 0"/>
             <geometry>
                 <mesh filename="package://oxbot_description/meshes/oxbot_front_wheel.stl" scale="0.001 0.001 0.001"/>
@@ -225,9 +224,8 @@
         </collision>
     </link>
-    <joint name="wheel_front_left_joint" type="continuous">
+    <joint name="wheel_front_left_joint" type="fixed">
         <parent link="chassis_bottom_link"/>
         <child link="wheel_front_left_link"/>
-        <axis xyz="1 0 0"/>
-        <origin rpy="0 0 0" xyz="-0.28 0.1325 0.026"/>
+        <origin rpy="0 0 0" xyz="0.1325 0.28 0.026"/>
     </joint>
     <link name="wheel_rear_right_link">
@@ -237,5 +235,5 @@
         </inertial>-->
         <visual>
-            <origin rpy="0 3.1415 0" xyz="0.105 0 0"/>
+            <origin rpy="0 0 1.57" xyz="0 -0.105 0"/>
             <geometry>
                 <mesh filename="package://oxbot_description/meshes/oxbot_rear_wheel.stl" scale="0.001 0.001 0.001"/>
@@ -249,9 +247,8 @@
         </collision>
     </link>
-    <joint name="wheel_rear_right_joint" type="continuous">
+    <joint name="wheel_rear_right_joint" type="fixed">
         <parent link="chassis_bottom_link"/>
         <child link="wheel_rear_right_link"/>
-        <axis xyz="1 0 0"/>
-        <origin rpy="0 0 0" xyz="0.28 -0.1325 0.049"/>
+        <origin rpy="0 0 0" xyz="-0.1325 -0.28 0.049"/>
     </joint>
     <link name="wheel_rear_left_link">
@@ -261,5 +258,5 @@
         </inertial>-->
         <visual>
-            <origin rpy="0 0 0" xyz="-0.105 0 0"/>
+            <origin rpy="0 0 -1.57" xyz="0 0.105 0"/>
             <geometry>
                 <mesh filename="package://oxbot_description/meshes/oxbot_rear_wheel.stl" scale="0.001 0.001 0.001"/>
@@ -273,9 +270,8 @@
         </collision>
     </link>
-    <joint name="wheel_rear_left_joint" type="continuous">
+    <joint name="wheel_rear_left_joint" type="fixed">
         <parent link="chassis_bottom_link"/>
         <child link="wheel_rear_left_link"/>
-        <axis xyz="1 0 0"/>
-        <origin rpy="0 0 0" xyz="-0.28 -0.1325 0.049"/>
+        <origin rpy="0 0 0" xyz="-0.1325 0.28 0.049"/>
     </joint>
 </robot>

Commit message: adjusting sensor frames

File: src/ros2_ws/src/oxbot_description/urdf/oxbot.urdf.xacro (robot description, xacro)
@@ -81,5 +81,5 @@
         </inertial>-->
         <visual>
-            <origin rpy="1.57 0 1.57" xyz="0 0 0"/>
+            <origin rpy="1.57 0 1.57" xyz="0.01 -0.055 0.01"/>
             <geometry>
                 <mesh filename="package://oxbot_description/meshes/d455.stl" scale="0.001 0.001 0.001"/>
@@ -88,7 +88,7 @@
     </link>
     <joint name="camera_joint" type="fixed">
-        <parent link="camera_mount_link"/>
+        <parent link="chassis_bottom_link"/>
         <child link="camera_link"/>
-        <origin rpy="0 0 0" xyz="-0.002 0 0.0325"/>
+        <origin rpy="0 0 0" xyz="0.08255 0.05318 0.2778125"/>
     </joint>
     <link name="lidar_link">
@@ -99,5 +99,5 @@
         </inertial>-->
         <visual>
-            <origin rpy="1.57 0 0" xyz="-0.0351 0.0351 -0.044"/>
+            <origin rpy="1.57 0 0" xyz="-0.0351 0.0351 -0.037"/>
             <geometry>
                 <mesh filename="package://oxbot_description/meshes/rplidar_main.STL" scale="0.001 0.001 0.001"/>
@@ -112,7 +112,7 @@
     </link>
     <joint name="lidar_joint" type="fixed">
-        <parent link="chassis_top_link"/>
+        <parent link="chassis_bottom_link"/>
         <child link="lidar_link"/>
-        <origin rpy="0 0 -1.57" xyz="0.015 -0.01 0.184"/>
+        <origin rpy="0 0 -1.57" xyz="0.0 0.0 0.29369"/>
     </joint>
     <link name="fan1_link">

Commit message: adding tags for gazebo sim

File: src/ros2_ws/src/oxbot_description/urdf/oxbot.urdf.xacro (robot description, xacro)
@@ -1,13 +1,10 @@
 <?xml version="1.0"?>
 <robot xmlns:xacro="http://www.ros.org/wiki/xacro" name="oxbot">
+    <xacro:include filename="$(find oxbot_description)/urdf/oxbot_gazebo.xacro"/>
     <link name="base_footprint"/>
     <link name="chassis_bottom_link">
-        <!--<inertial>
-            <origin xyz="0 0 0.0575" rpy="0.0 0.0 0.0"/>
-            <mass value="8"/>
-            <inertia ixx="9.330733e-02" iyy="2.1713733e-01" izz="2.92811333e-01"/>
-        </inertial>-->
-        <visual>
-            <origin rpy="0 0 -1.57" xyz="0 0 0"/>
+        <inertial auto="true" />
+        <visual>
+            <origin rpy="0 0 0" xyz="0 0 0"/>
             <geometry>
                 <mesh filename="package://oxbot_description/meshes/oxbot_chassis_bottom.stl" scale="0.001 0.001 0.001"/>
@@ -19,4 +16,5 @@
                 <mesh filename="package://oxbot_description/meshes/oxbot_chassis_bottom.stl" scale="0.001 0.001 0.001"/>
             </geometry>
+            <density>1000.0</density>
         </collision>
     </link>
@@ -27,11 +25,7 @@
     </joint>
     <link name="chassis_top_link">
-        <!--<inertial>
-            <origin xyz="0 0 0.0575" rpy="0.0 0.0 0.0"/>
-            <mass value="8"/>
-            <inertia ixx="9.330733e-02" iyy="2.1713733e-01" izz="2.92811333e-01"/>
-        </inertial>-->
-        <visual>
-            <origin rpy="0 0 -1.57" xyz="0 0 0"/>
+        <inertial auto="true" />
+        <visual>
+            <origin rpy="0 0 0" xyz="0 0 0"/>
             <geometry>
                 <mesh filename="package://oxbot_description/meshes/oxbot_chassis_top.stl" scale="0.001 0.001 0.001"/>
@@ -39,4 +33,5 @@
         </visual>
         <collision>
+            <density>333.0</density>
             <origin rpy="0 0 0" xyz="0 0 0"/>
             <geometry>
@@ -51,9 +46,5 @@
     </joint>
     <link name="camera_mount_link">
-        <!--<inertial>
-            <origin xyz="0 0 0.0575" rpy="0.0 0.0 0.0"/>
-            <mass value="8"/>
-            <inertia ixx="9.330733e-02" iyy="2.1713733e-01" izz="2.92811333e-01"/>
-        </inertial>-->
+        <inertial auto="true" />
         <visual>
             <origin rpy="0 0 1.57" xyz="0 -0.09 0"/> <!--xyz="0.09 0 0"/> -->
@@ -63,4 +54,5 @@
         </visual>
         <collision>
+            <density>250.0</density>
             <origin rpy="0 0 0" xyz="0 0 0"/>
             <geometry>
@@ -75,9 +67,5 @@
     </joint>
     <link name="camera_link">
-        <!--<inertial>
-            <origin xyz="0 0 0.0575" rpy="0.0 0.0 0.0"/>
-            <mass value="8"/>
-            <inertia ixx="9.330733e-02" iyy="2.1713733e-01" izz="2.92811333e-01"/>
-        </inertial>-->
+        <inertial auto="true" />
         <visual>
             <origin rpy="1.57 0 1.57" xyz="0.01 -0.055 0.01"/>
@@ -86,4 +74,11 @@
             </geometry>
         </visual>
+        <collision>
+            <density>1000.0</density>
+            <origin rpy="0 0 0" xyz="0 0 0 "/>
+            <geometry>
+                <box size="0.18 0.03 0.04"/>
+            </geometry>
+        </collision>
     </link>
     <joint name="camera_joint" type="fixed">
@@ -93,9 +88,5 @@
     </joint>
     <link name="lidar_link">
-        <!--<inertial>
-            <origin xyz="0 0 0.0575" rpy="0.0 0.0 0.0"/>
-            <mass value="8"/>
-            <inertia ixx="9.330733e-02" iyy="2.1713733e-01" izz="2.92811333e-01"/>
-        </inertial>-->
+        <inertial auto="true" />
         <visual>
             <origin rpy="1.57 0 0" xyz="-0.0351 0.0351 -0.037"/>
@@ -105,4 +96,5 @@
         </visual>
         <collision>
+            <density>750.0</density>
             <origin rpy="0 0 0" xyz="0 0 0"/>
             <geometry>
@@ -117,17 +109,14 @@
     </joint>
     <link name="fan1_link">
-        <!--<inertial>
-            <origin xyz="0 0 0.0575" rpy="0.0 0.0 0.0"/>
-            <mass value="8"/>
-            <inertia ixx="9.330733e-02" iyy="2.1713733e-01" izz="2.92811333e-01"/>
-        </inertial>-->
-        <visual>
-            <origin rpy="0 0 0" xyz="0 0 0"/>
-            <geometry>
-                <mesh filename="package://oxbot_description/meshes/oxbot_fan.stl" scale="0.001 0.001 0.001"/>
-            </geometry>
-        </visual>
-        <collision>
-            <origin rpy="0 0 0" xyz="0 0 0"/>
+        <inertial auto="true" />
+        <visual>
+            <origin rpy="0 0 0" xyz="0 0 0"/>
+            <geometry>
+                <mesh filename="package://oxbot_description/meshes/oxbot_fan.stl" scale="0.001 0.001 0.001"/>
+            </geometry>
+        </visual>
+        <collision>
+            <density>500.0</density>
+            <origin rpy="0 0 0" xyz="-0.121 0 0"/>
             <geometry>
                 <mesh filename="package://oxbot_description/meshes/oxbot_fan.stl" scale="0.001 0.001 0.001"/>
@@ -141,9 +130,5 @@
     </joint>
     <link name="fan2_link">
-        <!--<inertial>
-            <origin xyz="0 0 0.0575" rpy="0.0 0.0 0.0"/>
-            <mass value="8"/>
-            <inertia ixx="9.330733e-02" iyy="2.1713733e-01" izz="2.92811333e-01"/>
-        </inertial>-->
+        <inertial auto="true" />
         <visual>
             <origin rpy="0 0 0" xyz="-0 0 0"/>
@@ -153,5 +138,6 @@
         </visual>
         <collision>
-            <origin rpy="0 0 0" xyz="0 0 0"/>
+            <density>500.0</density>
+            <origin rpy="0 0 0" xyz="-0.121 0 0"/>
             <geometry>
                 <mesh filename="package://oxbot_description/meshes/oxbot_fan.stl" scale="0.001 0.001 0.001"/>
@@ -165,4 +151,5 @@
     </joint>
     <link name="antenna_link">
+        <inertial auto="true" />
         <visual>
             <origin rpy="0 0 0" xyz="0 0 0"/>
@@ -172,4 +159,5 @@
         </visual>
         <collision>
+            <density>750.0</density>
             <origin rpy="0 0 0" xyz="0 0 0"/>
             <geometry>
@@ -184,8 +172,5 @@
     </joint>
     <link name="wheel_front_right_link">
-        <!--<inertial>
-            <mass value="3"/>
-            <inertia ixx="6.7775e-01" iyy="6.7775e-01" izz="1.35375e-02"/>
-        </inertial>-->
+        <inertial auto="true" />
         <visual>
             <origin rpy="0 0 01.57" xyz="0 -0.075 0"/>
@@ -195,4 +180,5 @@
         </visual>
         <collision>
+            <density>6000.0</density>
             <origin xyz="0.075 0 0" rpy="0 0 0"/>
             <geometry>
@@ -201,14 +187,12 @@
         </collision>
     </link>
-    <joint name="wheel_front_right_joint" type="fixed">
+    <joint name="wheel_front_right_joint" type="continuous">
         <parent link="chassis_bottom_link"/>
         <child link="wheel_front_right_link"/>
+        <axis xyz="0 1 0"/>
         <origin rpy="0 0 0" xyz="0.1325 -0.28 0.026"/>
     </joint>
     <link name="wheel_front_left_link">
-        <!--<inertial>
-            <mass value="3"/>
-            <inertia ixx="6.7775e-01" iyy="6.7775e-01" izz="1.35375e-02"/>
-        </inertial>-->
+        <inertial auto="true" />
         <visual>
             <origin rpy="0 0 -1.57" xyz="0 0.075 0"/>
@@ -218,4 +202,5 @@
         </visual>
         <collision>
+            <density>6000.0</density>
             <origin xyz="-0.075 0 0" rpy="0 0 0"/>
             <geometry>
@@ -224,14 +209,12 @@
         </collision>
     </link>
-    <joint name="wheel_front_left_joint" type="fixed">
+    <joint name="wheel_front_left_joint" type="continuous">
         <parent link="chassis_bottom_link"/>
         <child link="wheel_front_left_link"/>
+        <axis xyz="0 1 0"/>
         <origin rpy="0 0 0" xyz="0.1325 0.28 0.026"/>
     </joint>
     <link name="wheel_rear_right_link">
-        <!--<inertial>
-            <mass value="3"/>
-            <inertia ixx="6.7775e-01" iyy="6.7775e-01" izz="1.35375e-02"/>
-        </inertial>-->
+        <inertial auto="true" />
         <visual>
             <origin rpy="0 0 1.57" xyz="0 -0.105 0"/>
@@ -241,4 +224,5 @@
         </visual>
         <collision>
+            <density>6000.0</density>
             <origin xyz="0 0 0" rpy="0 0 0"/>
             <geometry>
@@ -247,14 +231,12 @@
         </collision>
     </link>
-    <joint name="wheel_rear_right_joint" type="fixed">
+    <joint name="wheel_rear_right_joint" type="continuous">
         <parent link="chassis_bottom_link"/>
         <child link="wheel_rear_right_link"/>
+        <axis xyz="0 1 0"/>
         <origin rpy="0 0 0" xyz="-0.1325 -0.28 0.049"/>
     </joint>
     <link name="wheel_rear_left_link">
-        <!--<inertial>
-            <mass value="3"/>
-            <inertia ixx="6.7775e-01" iyy="6.7775e-01" izz="1.35375e-02"/>
-        </inertial>-->
+        <inertial auto="true" />
         <visual>
             <origin rpy="0 0 -1.57" xyz="0 0.105 0"/>
@@ -264,4 +246,5 @@
         </visual>
         <collision>
+            <density>6000.0</density>
             <origin xyz="0 0 0" rpy="0 0 0"/>
             <geometry>
@@ -270,7 +253,8 @@
         </collision>
     </link>
-    <joint name="wheel_rear_left_joint" type="fixed">
+    <joint name="wheel_rear_left_joint" type="continuous">
         <parent link="chassis_bottom_link"/>
         <child link="wheel_rear_left_link"/>
+        <axis xyz="0 1 0"/>
         <origin rpy="0 0 0" xyz="-0.1325 0.28 0.049"/>
     </joint>

File: src/ros2_ws/src/oxbot_description/urdf/oxbot_gazebo.xacro (robot description, xacro)
@@ -1,5 +1,41 @@
 <?xml version="1.0"?>
 <robot name="oxbot" xmlns:xacro="http://www.ros.org/wiki/xacro">
-    <transmission name="wheel_front_right_transmission">
+    <gazebo reference="wheel_front_right_link">
+		<mu1>100000000000000.0</mu1>
+		<mu2>100000000000000.0</mu2>
+		<kp>1000000000000.0</kp>
+		<kd>10.0</kd>
+		<minDepth>0.001</minDepth>
+		<maxVal>0.1</maxVal>
+		<fdir1>1 0 0</fdir1>
+	</gazebo>
+	<gazebo reference="wheel_front_left_link">
+		<mu1>100000000000000.0</mu1>
+		<mu2>100000000000000.0</mu2>
+		<kp>1000000000000.0</kp>
+		<kd>10.0</kd>
+		<minDepth>0.001</minDepth>
+		<maxVal>0.1</maxVal>
+		<fdir1>1 0 0</fdir1>
+	</gazebo>
+	<gazebo reference="wheel_rear_left_link">
+		<mu1>100000000000000.0</mu1>
+		<mu2>100000000000000.0</mu2>
+		<kp>1000000000000.0</kp>
+		<kd>10.0</kd>
+		<minDepth>0.001</minDepth>
+		<maxVal>0.1</maxVal>
+		<fdir1>1 0 0</fdir1>
+	</gazebo>
+	<gazebo reference="wheel_rear_right_link">
+		<mu1>100000000000000.0</mu1>
+		<mu2>100000000000000.0</mu2>
+		<kp>1000000000000.0</kp>
+		<kd>10.0</kd>
+		<minDepth>0.001</minDepth>
+		<maxVal>0.1</maxVal>
+		<fdir1>1 0 0</fdir1>
+	</gazebo>
+    <!-- <transmission name="wheel_front_right_transmission">
         <plugin>transmission_interface/SimpleTransmission</plugin>
         <actuator name="wheel_front_right_motor" role="actuator_front_right"/>
@@ -7,4 +43,4 @@
             <mechanical_reduction>1.0</mechanical_reduction>
         </joint>
-    </transmission>
+    </transmission> -->
 </robot>
