Commit message: working on adding gazebo sim

File: src/ros2_ws/src/oxbot_description/urdf/oxbot.urdf.xacro (robot description, xacro)
@@ -4,5 +4,9 @@
     <link name="base_footprint"/>
     <link name="chassis_bottom_link">
-        <inertial auto="true" />
+        <inertial>
+            <origin rpy="0 0 0" xyz="0 0 0.0575"/>
+            <mass value="4.5"/>
+            <inertia ixx="0.12205" ixy="0.0" ixz="0.0" iyy="0.05243" iyz="0.0" izz="0.16467"/>
+        </inertial>
         <visual>
             <origin rpy="0 0 0" xyz="0 0 0"/>
@@ -16,5 +20,4 @@
                 <mesh filename="package://oxbot_description/meshes/oxbot_chassis_bottom.stl" scale="0.001 0.001 0.001"/>
             </geometry>
-            <density>1000.0</density>
         </collision>
     </link>
@@ -25,5 +28,9 @@
     </joint>
     <link name="chassis_top_link">
-        <inertial auto="true" />
+        <inertial>
+            <origin rpy="0 0 0" xyz="0 0 0.07"/>
+            <mass value="2.0"/>
+            <inertia ixx="0.05553" ixy="0.0" ixz="0.0" iyy="0.01208" iyz="0.0" izz="0.06108"/>
+        </inertial>
         <visual>
             <origin rpy="0 0 0" xyz="0 0 0"/>
@@ -33,5 +40,4 @@
         </visual>
         <collision>
-            <density>333.0</density>
             <origin rpy="0 0 0" xyz="0 0 0"/>
             <geometry>
@@ -46,7 +52,11 @@
     </joint>
     <link name="camera_mount_link">
-        <inertial auto="true" />
-        <visual>
-            <origin rpy="0 0 1.57" xyz="0 -0.09 0"/> <!--xyz="0.09 0 0"/> -->
+        <inertial>
+            <origin rpy="0 0 0" xyz="0 0 0"/>
+            <mass value="0.1"/>
+            <inertia ixx="0.000283" ixy="0.0" ixz="0.0" iyy="0.000020" iyz="0.0" izz="0.00027"/>
+        </inertial>
+        <visual>
+            <origin rpy="0 0 1.57" xyz="0 -0.09 0"/>
             <geometry>
                 <mesh filename="package://oxbot_description/meshes/oxbot_realsense_mount.stl" scale="0.001 0.001 0.001"/>
@@ -54,5 +64,4 @@
         </visual>
         <collision>
-            <density>250.0</density>
             <origin rpy="0 0 0" xyz="0 0 0"/>
             <geometry>
@@ -67,5 +76,9 @@
     </joint>
     <link name="camera_link">
-        <inertial auto="true" />
+        <inertial>
+            <origin rpy="0 0 0" xyz="0 0 0"/>
+            <mass value="0.072" />
+            <inertia ixx="0.003881243" ixy="0.0" ixz="0.0" iyy="0.000498940" iyz="0.0" izz="0.003879257" />
+        </inertial>
         <visual>
             <origin rpy="1.57 0 1.57" xyz="0.01 -0.055 0.01"/>
@@ -75,5 +88,4 @@
         </visual>
         <collision>
-            <density>1000.0</density>
             <origin rpy="0 0 0" xyz="0 0 0 "/>
             <geometry>
@@ -88,5 +100,9 @@
     </joint>
     <link name="lidar_link">
-        <inertial auto="true" />
+        <inertial>
+            <origin rpy="0 0 0" xyz="0 0 0"/>
+            <mass value="0.17" />
+            <inertia ixx="1e-6" ixy="0" ixz="0" iyy="1e-6" iyz="0" izz="1e-6" />
+        </inertial>
         <visual>
             <origin rpy="1.57 0 0" xyz="-0.0351 0.0351 -0.037"/>
@@ -96,5 +112,4 @@
         </visual>
         <collision>
-            <density>750.0</density>
             <origin rpy="0 0 0" xyz="0 0 0"/>
             <geometry>
@@ -109,13 +124,16 @@
     </joint>
     <link name="fan1_link">
-        <inertial auto="true" />
-        <visual>
-            <origin rpy="0 0 0" xyz="0 0 0"/>
-            <geometry>
-                <mesh filename="package://oxbot_description/meshes/oxbot_fan.stl" scale="0.001 0.001 0.001"/>
-            </geometry>
-        </visual>
-        <collision>
-            <density>500.0</density>
+        <inertial>
+            <origin rpy="0 0 0" xyz="0 0 0"/>
+            <mass value="0.05" />
+            <inertia ixx="63e-6" ixy="0" ixz="0" iyy="63e-6" iyz="0" izz="122e-6" />
+        </inertial>
+        <visual>
+            <origin rpy="0 0 0" xyz="0 0 0"/>
+            <geometry>
+                <mesh filename="package://oxbot_description/meshes/oxbot_fan.stl" scale="0.001 0.001 0.001"/>
+            </geometry>
+        </visual>
+        <collision>
             <origin rpy="0 0 0" xyz="-0.121 0 0"/>
             <geometry>
@@ -130,5 +148,9 @@
     </joint>
     <link name="fan2_link">
-        <inertial auto="true" />
+        <inertial>
+            <origin rpy="0 0 0" xyz="0 0 0"/>
+            <mass value="0.05" />
+            <inertia ixx="63e-6" ixy="0" ixz="0" iyy="63e-6" iyz="0" izz="122e-6" />
+        </inertial>
         <visual>
             <origin rpy="0 0 0" xyz="-0 0 0"/>
@@ -138,5 +160,4 @@
         </visual>
         <collision>
-            <density>500.0</density>
             <origin rpy="0 0 0" xyz="-0.121 0 0"/>
             <geometry>
@@ -151,5 +172,9 @@
     </joint>
     <link name="antenna_link">
-        <inertial auto="true" />
+        <inertial>
+            <origin rpy="0 0 0" xyz="0 0 0"/>
+            <mass value="0.025" />
+            <inertia ixx="1e-6" ixy="0" ixz="0" iyy="1e-6" iyz="0" izz="1e-6" />
+        </inertial>
         <visual>
             <origin rpy="0 0 0" xyz="0 0 0"/>
@@ -159,5 +184,4 @@
         </visual>
         <collision>
-            <density>750.0</density>
             <origin rpy="0 0 0" xyz="0 0 0"/>
             <geometry>
@@ -172,5 +196,9 @@
     </joint>
     <link name="wheel_front_right_link">
-        <inertial auto="true" />
+        <inertial>
+            <origin rpy="0 0 0" xyz="0 0 0"/>
+            <mass value="3.0" />
+            <inertia ixx="0.005772" ixy="0" ixz="0" iyy="0.010086" iyz="0" izz="0.005772" />
+        </inertial>
         <visual>
             <origin rpy="0 0 01.57" xyz="0 -0.075 0"/>
@@ -180,5 +208,4 @@
         </visual>
         <collision>
-            <density>6000.0</density>
             <origin xyz="0.075 0 0" rpy="0 0 0"/>
             <geometry>
@@ -194,5 +221,9 @@
     </joint>
     <link name="wheel_front_left_link">
-        <inertial auto="true" />
+        <inertial>
+            <origin rpy="0 0 0" xyz="0 0 0"/>
+            <mass value="3.0" />
+            <inertia ixx="0.005772" ixy="0" ixz="0" iyy="0.010086" iyz="0" izz="0.005772" />
+        </inertial>
         <visual>
             <origin rpy="0 0 -1.57" xyz="0 0.075 0"/>
@@ -202,5 +233,4 @@
         </visual>
         <collision>
-            <density>6000.0</density>
             <origin xyz="-0.075 0 0" rpy="0 0 0"/>
             <geometry>
@@ -216,5 +246,9 @@
     </joint>
     <link name="wheel_rear_right_link">
-        <inertial auto="true" />
+        <inertial>
+            <origin rpy="0 0 0" xyz="0 0 0"/>
+            <mass value="4.0" />
+            <inertia ixx="0.014425" ixy="0" ixz="0" iyy="0.02645" iyz="0" izz="0.014425" />
+        </inertial>
         <visual>
             <origin rpy="0 0 1.57" xyz="0 -0.105 0"/>
@@ -224,5 +258,4 @@
         </visual>
         <collision>
-            <density>6000.0</density>
             <origin xyz="0 0 0" rpy="0 0 0"/>
             <geometry>
@@ -238,5 +271,9 @@
     </joint>
     <link name="wheel_rear_left_link">
-        <inertial auto="true" />
+        <inertial>
+            <origin rpy="0 0 0" xyz="0 0 0"/>
+            <mass value="4.0" />
+            <inertia ixx="0.014425" ixy="0" ixz="0" iyy="0.02645" iyz="0" izz="0.014425" />
+        </inertial>
         <visual>
             <origin rpy="0 0 -1.57" xyz="0 0.105 0"/>
@@ -246,5 +283,4 @@
         </visual>
         <collision>
-            <density>6000.0</density>
             <origin xyz="0 0 0" rpy="0 0 0"/>
             <geometry>

Commit message: fixed URDF

File: src/ros2_ws/src/oxbot_description/urdf/oxbot.urdf.xacro (robot description, xacro)
@@ -10,5 +10,5 @@
         </inertial>
         <visual>
-            <origin rpy="0 0 0" xyz="0 0 0"/>
+            <origin rpy="0 0 -1.57" xyz="0 0 0"/>
             <geometry>
                 <mesh filename="package://oxbot_description/meshes/oxbot_chassis_bottom.stl" scale="0.001 0.001 0.001"/>
@@ -34,5 +34,5 @@
         </inertial>
         <visual>
-            <origin rpy="0 0 0" xyz="0 0 0"/>
+            <origin rpy="0 0 -1.57" xyz="0 0 0"/>
             <geometry>
                 <mesh filename="package://oxbot_description/meshes/oxbot_chassis_top.stl" scale="0.001 0.001 0.001"/>

Commit message: fixing URDF collision tags

File: src/ros2_ws/src/oxbot_description/urdf/oxbot.urdf.xacro (robot description, xacro)
@@ -208,5 +208,5 @@
         </visual>
         <collision>
-            <origin xyz="0.075 0 0" rpy="0 0 0"/>
+            <origin rpy="0 0 01.57" xyz="0 -0.075 0"/>
             <geometry>
                 <mesh filename="package://oxbot_description/meshes/oxbot_front_wheel.stl" scale="0.001 0.001 0.001"/>
@@ -233,5 +233,5 @@
         </visual>
         <collision>
-            <origin xyz="-0.075 0 0" rpy="0 0 0"/>
+            <origin rpy="0 0 -1.57" xyz="0 0.075 0"/>
             <geometry>
                 <mesh filename="package://oxbot_description/meshes/oxbot_front_wheel.stl" scale="0.001 0.001 0.001"/>
@@ -258,5 +258,5 @@
         </visual>
         <collision>
-            <origin xyz="0 0 0" rpy="0 0 0"/>
+            <origin rpy="0 0 1.57" xyz="0 -0.105 0"/>
             <geometry>
                 <mesh filename="package://oxbot_description/meshes/oxbot_rear_wheel.stl" scale="0.001 0.001 0.001"/>
@@ -283,5 +283,5 @@
         </visual>
         <collision>
-            <origin xyz="0 0 0" rpy="0 0 0"/>
+            <origin rpy="0 0 -1.57" xyz="0 0.105 0"/>
             <geometry>
                 <mesh filename="package://oxbot_description/meshes/oxbot_rear_wheel.stl" scale="0.001 0.001 0.001"/>

Commit message: added joystick to gazebo sim

File: src/ros2_ws/src/oxbot_description/urdf/oxbot.urdf.xacro (robot description, xacro)
@@ -18,5 +18,5 @@
         </visual>
         <collision>
-            <origin rpy="0 0 0" xyz="0 0 0"/>
+            <origin rpy="0 0 -1.57" xyz="0 0 0"/>
             <geometry>
                 <mesh filename="package://oxbot_description/meshes/oxbot_chassis_bottom.stl" scale="0.001 0.001 0.001"/>
@@ -42,5 +42,5 @@
         </visual>
         <collision>
-            <origin rpy="0 0 0" xyz="0 0 0"/>
+            <origin rpy="0 0 -1.57" xyz="0 0 0"/>
             <geometry>
                 <mesh filename="package://oxbot_description/meshes/oxbot_chassis_top.stl" scale="0.001 0.001 0.001"/>
@@ -66,5 +66,5 @@
         </visual>
         <collision>
-            <origin rpy="0 0 0" xyz="0 0 0"/>
+            <origin rpy="0 0 1.57" xyz="0 0 0"/>
             <geometry>
                 <box size="0.180 0.03 0.04"/>
@@ -90,5 +90,5 @@
         </visual>
         <collision>
-            <origin rpy="0 0 0" xyz="0 0 0 "/>
+            <origin rpy="1.57 0 1.57" xyz="0.01 -0.055 0.01"/>
             <geometry>
                 <box size="0.18 0.03 0.04"/>
@@ -114,5 +114,5 @@
         </visual>
         <collision>
-            <origin rpy="0 0 0" xyz="0 0 0"/>
+            <origin rpy="1.57 0 0" xyz="0 0 0"/>
             <geometry>
                 <box size="0.110 0.09 0.09"/>
@@ -138,5 +138,5 @@
         </visual>
         <collision>
-            <origin rpy="0 0 0" xyz="-0.121 0 0"/>
+            <origin rpy="0 0 0" xyz="0 0 0"/>
             <geometry>
                 <mesh filename="package://oxbot_description/meshes/oxbot_fan.stl" scale="0.001 0.001 0.001"/>
@@ -162,5 +162,5 @@
         </visual>
         <collision>
-            <origin rpy="0 0 0" xyz="-0.121 0 0"/>
+            <origin rpy="0 0 0" xyz="-0 0 0"/>
             <geometry>
                 <mesh filename="package://oxbot_description/meshes/oxbot_fan.stl" scale="0.001 0.001 0.001"/>

Commit message: initial cartographer .lua config added

File: src/ros2_ws/src/oxbot_description/urdf/oxbot.urdf.xacro (robot description, xacro)
@@ -17,5 +17,6 @@
             </geometry>
         </visual>
-        <collision>
+        <collision>  map_builder = MAP_BUILDER,
+  trajectory_builder = TRAJECTORY_BUILDER,
             <origin rpy="0 0 -1.57" xyz="0 0 0"/>
             <geometry>

Commit message: configuring cartographer options

File: src/ros2_ws/src/oxbot_description/urdf/oxbot.urdf.xacro (robot description, xacro)
@@ -17,6 +17,5 @@
             </geometry>
         </visual>
-        <collision>  map_builder = MAP_BUILDER,
-  trajectory_builder = TRAJECTORY_BUILDER,
+        <collision>
             <origin rpy="0 0 -1.57" xyz="0 0 0"/>
             <geometry>

Commit message: moved lidar frame +z

File: src/ros2_ws/src/oxbot_description/urdf/oxbot.urdf.xacro (robot description, xacro)
@@ -108,5 +108,5 @@
         </inertial>
         <visual>
-            <origin rpy="1.57 0 0" xyz="-0.0351 0.0351 -0.037"/>
+            <origin rpy="1.57 0 0" xyz="-0.0351 0.0351 -0.06415"/>
             <geometry>
                 <mesh filename="package://oxbot_description/meshes/rplidar_main.STL" scale="0.001 0.001 0.001"/>
@@ -123,5 +123,5 @@
         <parent link="chassis_bottom_link"/>
         <child link="lidar_link"/>
-        <origin rpy="0 0 -1.57" xyz="0.0 0.0 0.29369"/>
+        <origin rpy="0 0 -1.57" xyz="0.0 0.0 0.3208"/>
     </joint>
     <link name="fan1_link">
